Commit message: attached urdf progress

File: bin/resources/jumping_panda.urdf (robot description, URDF)
Before this commit: robot mmp_panda, 14 links, 13 joints
Links:
- removed link leg_left_upper
- added link LL_KOSY_L1, mass 2.7752200000; visual mesh filename=../../model/toro/meshes/obj/left_lower_hip.stl.obj
- added link LL_KOSY_L23, mass 2.2450500000; visual mesh filename=../../model/toro/meshes/obj/kuka-link2.stl.obj
- added link LL_KOSY_L4, mass 2.6274500000; visual mesh filename=../../model/toro/meshes/obj/kuka-link3.stl.obj
- added link LL_KOSY_L56, mass 5.7035400000; visual mesh filename=../../model/toro/meshes/obj/left_calf.stl.obj
- added link RL_KOSY_L1, mass 2.7752200000; visual mesh filename=../../model/toro/meshes/obj/right_lower_hip.stl.obj
- added link RL_KOSY_L23, mass 2.2450500000; visual mesh filename=../../model/toro/meshes/obj/kuka-link2.stl.obj
- added link RL_KOSY_L4, mass 2.6274500000; visual mesh filename=../../model/toro/meshes/obj/kuka-link3.stl.obj
- added link RL_KOSY_L56, mass 5.7035400000; visual mesh filename=../../model/toro/meshes/obj/right_calf.stl.obj
- link base_link: geometry collision box size=0.5 0.5 0.5
Joints:
- removed joint joint_leg_left_upper
- added joint joint_leg_left1: type fixed, parent base_link, child LL_KOSY_L1, origin xyz=0.0000000000 0.1000000000 0.1 rpy=0 0 0, axis  1 0 0 , limit lower=-0.7804 upper=1.5708 effort=176 velocity=1.9199
- added joint joint_leg_left2: type revolute, parent LL_KOSY_L1, child LL_KOSY_L23, origin xyz=0.0000000000 0.0350000000 -0.1200000000 rpy=0 0 0, axis 0 1 0, limit lower=-2.0071 upper=1.5708 effort=100 velocity=2.7402
- added joint joint_leg_left3: type fixed, parent LL_KOSY_L23, child LL_KOSY_L4, axis 0 0 1, limit lower=-2.0944 upper=2.0944 effort=100 velocity=2.7402
- added joint joint_leg_left4: type revolute, parent LL_KOSY_L4, child LL_KOSY_L56, origin xyz=0.0000000000 0.0000000000 -0.3999000880 rpy=0 0 0, axis 0 1 0, limit lower=-1.8326 upper=1.8326 effort=165 velocity=3.0718
- added joint joint_leg_right1: type fixed, parent base_link, child RL_KOSY_L1, origin xyz=-0.0000000000 -0.1000000000 0.1 rpy=0 0 0, axis 1 0 0, limit lower=-1.5708 upper=0.7854 effort=176 velocity=1.9199
- added joint joint_leg_right2: type revolute, parent RL_KOSY_L1, child RL_KOSY_L23, origin xyz=-0.0000000000 -0.0350000000 -0.1200000000 rpy=0 0 0, axis 0 1 0, limit lower=-2.0071 upper=1.5708 effort=100 velocity=2.7402
- added joint joint_leg_right3: type fixed, parent RL_KOSY_L23, child RL_KOSY_L4, axis 0 0 1, limit lower=-2.0944 upper=2.0944 effort=100 velocity=2.7402
- added joint joint_leg_right4: type revolute, parent RL_KOSY_L4, child RL_KOSY_L56, origin xyz=0.0000000000 0.0000000000 -0.3999000880 rpy=0 0 0, axis 0 1 0, limit lower=-1.8326 upper=1.8326 effort=165 velocity=3.0718
