Commit message: simulation setup

File: mmp_panda.urdf (robot description, URDF)
Before this commit: robot mmp_panda, 12 links, 11 joints
Links:
- link base_link: geometry visual mesh filename=../../model/mmp_panda/meshes/panda_BaseCombo.obj
- link link1: geometry visual mesh filename=../../model/panda/meshes/visual/link1.obj
- link link2: geometry visual mesh filename=../../model/panda/meshes/visual/link2.obj
- link link3: geometry visual mesh filename=../../model/panda/meshes/visual/link3.obj
- link link4: geometry visual mesh filename=../../model/panda/meshes/visual/link4.obj
- link link5: geometry visual mesh filename=../../model/panda/meshes/visual/link5.obj
- link link6: geometry visual mesh filename=../../model/panda/meshes/visual/link6.obj
- link link7: geometry visual mesh filename=../../model/panda/meshes/visual/link7.obj
- link racquetlink: geometry collision box size=0.25 1.5 0.0002; visual mesh filename=../../Objects/Visual/TennisRacquet.obj

Commit message: New files for Panda robot and new simviz to run the world

File: mmp_panda.urdf (robot description, URDF)
Before this commit: robot mmp_panda, 12 links, 11 joints
Links:
- removed link racquetlink
- link link7: mass 0.03268873 -> 3.0; geometry visual box size=0.15 0.15 0.01; visual mesh filename=../../model/panda/meshes/visual/link7.obj
Joints:
- removed joint joint8
- joint base_prismatic_x: limit effort=0 velocity=2.0 -> lower=-2.8973 upper=2.9873 effort=87 velocity=2.1750
- joint base_prismatic_y: limit effort=0 velocity=2.0 -> lower=-2.8973 upper=2.9873 effort=87 velocity=2.1750
- joint joint1: limit lower=-2.8973 upper=2.8973 effort=100 velocity=100.0 -> lower=-2.8973 upper=2.8973 effort=87 velocity=2.1750

Commit message: Collision meshes added to net, end effector size adjusted and collision added, ball collision adjusted. Still need to add posts

File: mmp_panda.urdf (robot description, URDF)
Before this commit: robot mmp_panda, 11 links, 10 joints
Links:
- link link7: geometry collision box size=0.25 0.25 0.01; visual box size=0.25 0.25 0.01
