Commit message: simple bounce demo

File: legged_panda.urdf (robot description, URDF)
Before this commit: robot mmp_panda, 21 links, 20 joints
Links:
- added link LL_foot, mass 1.5; collision box size=0.2 0.2 0.05; visual box size=0.2 0.2 0.05
- added link RL_foot, mass 1.5; collision box size=0.2 0.2 0.05; visual box size=0.2 0.2 0.05
- link racquetlink: geometry collision box size=0.25 0.25 0.05; visual box size=0.25 0.25 0.05
Joints:
- added joint joint_leg_left5: type revolute, parent LL_KOSY_L56, child LL_foot, origin xyz=0.0000000000 0.0000000000 -0.3999000880 rpy=0 0 0, axis 0 1 0, limit lower=-1.8326 upper=1.8326 effort=165 velocity=3.0718
- added joint joint_leg_right5: type revolute, parent RL_KOSY_L56, child RL_foot, origin xyz=0.0000000000 0.0000000000 -0.3999000880 rpy=0 0 0, axis 0 1 0, limit lower=-1.8326 upper=1.8326 effort=165 velocity=3.0718

File: simple_legged_panda.urdf (robot description, URDF)
Before this commit: robot mmp_panda, 18 links, 17 joints
Links:
- link racquetlink: geometry collision box size=0.25 1.5 0.0002; visual origin xyz=0.2 0 0
Joints:
- joint joint_leg_left2: origin xyz=0.0000000000 -0.0350000000 0.1200000000 rpy=0 0 0 -> xyz=0.0000000000 -0.0350000000 0.43 rpy=0 0 0
- joint joint_leg_left4: origin xyz=0.0000000000 0.0000000000 0.3999000880 rpy=0 0 0 -> xyz=0.0000000000 0.0000000000 0.0 rpy=0 0 0

Commit message: progress on posture control

File: legged_panda.urdf (robot description, URDF)
Before this commit: robot mmp_panda, 23 links, 22 joints
Links:
- link base_link: mass 64.6 -> 5.6

Commit message: base control progress

File: legged_panda.urdf (robot description, URDF)
Before this commit: robot mmp_panda, 23 links, 22 joints
Joints:
- joint base_prismatic_x: limit effort=0 velocity=2.0 -> effort=0 velocity=10.0
- joint base_prismatic_y: limit effort=0 velocity=2.0 -> effort=0 velocity=10.0
