Commit message: control progress

File: model/legged_panda.urdf (robot description, URDF)
Before this commit: robot mmp_panda, 22 links, 21 joints
Joints:
- joint joint1: limit lower=-2.8973 upper=2.8973 effort=100 velocity=100.0 -> lower=-2.8973 upper=2.8973 effort=1000 velocity=100.0
- joint joint2: limit lower=-1.7628 upper=1.7628 effort=87 velocity=2.1750 -> lower=-1.7628 upper=1.7628 effort=1000 velocity=2.1750
- joint joint3: limit lower=-2.8973 upper=2.8973 effort=87 velocity=2.1750 -> lower=-2.8973 upper=2.8973 effort=1000 velocity=2.1750
- joint joint4: limit lower=-3.0718 upper=-0.0698 effort=87 velocity=2.1750 -> lower=-3.0718 upper=-0.0698 effort=1000 velocity=2.1750
